File: a2audio/A2_Audio_Rev1/A2_Audio_Rev1.kicad_pcb (KiCad board)
At the start: 4 copper layers, 0 parts

Commit message: Added the new kicad footprints for each schematic, that didn't have one previously (most of them).
Parts:
- added D2: BAT54C, Package_TO_SOT_SMD:SOT-23, F.Cu at (106.0, 94.4)
- added D3: PMEG2020EH, Diode_SMD:D_SOD-123F, F.Cu at (116.6, 100.3)
- added D4: PMEG2020EH, Diode_SMD:D_SOD-123F, F.Cu at (116.6, 103.7)
- added IC1: ES9822QPRO, custom:QFN40P500X500X80-41N-D, F.Cu at (130.6, 113.9)
- added U1: USBLC6-2SC6, Package_TO_SOT_SMD:SOT-23-6, F.Cu at (122.4, 108.0)
- added U10: OPA1622IDRCR, custom:IC_OPA1622IDRCR, F.Cu at (172.8, 61.4)
- added U11: SI4732-A10-GS, custom:SOIC_A10-GS_SIL, F.Cu at (131.2, 104.5)
- added U12: OPA1612AIDR, custom:SOIC127P599X175-8N, F.Cu at (140.3, 111.1)
- added U13: LT3042xMSE, Package_SO:MSOP-10-1EP_3x3mm_P0.5mm_EP1.68x1.88mm, F.Cu at (107.2, 122.3)
- added U14: W25Q16JVSS, Package_SO:SOIC-8_5.3x5.3mm_P1.27mm, F.Cu at (108.7, 102.2)
- added U15: CM5108000, custom:MODULE_CM5108000, F.Cu at (131.8, 71.5)
- added U16: AP2112K-3.3, Package_TO_SOT_SMD:SOT-23-5, F.Cu at (138.1, 101.1)
- added U17: AP2112K-1.8, Package_TO_SOT_SMD:SOT-23-5, F.Cu at (138.1, 105.7)
- added U18: LT6711A, custom:QFN40P750X750X80-65N-D, F.Cu at (151.4, 103.6)
- added U19: TPS62130, Package_DFN_QFN:VQFN-16-1EP_3x3mm_P0.5mm_EP1.68x1.68mm_ThermalVias, F.Cu at (121.7, 120.9)
- added U2: TPS65987DDHRSHR, custom:IC_TPS65987DDHRSHR, F.Cu at (108.5, 110.1)
- added U20: AP2112K-1.8, Package_TO_SOT_SMD:SOT-23-5, F.Cu at (158.9, 101.1)
- added U21: TPS61230DRC, Package_SON:Texas_S-PVSON-N10_ThermalVias, F.Cu at (122.0, 101.3)
- added U22: AP2112K-1.2, Package_TO_SOT_SMD:SOT-23-5, F.Cu at (158.9, 105.7)
- added U23: LTC2954ITS8-1_TRPBF, custom:TSOT-23_TS8, F.Cu at (110.7, 94.4)
- added U24: TPS65131RGE, Package_DFN_QFN:VQFN-24-1EP_4x4mm_P0.5mm_EP2.45x2.45mm_ThermalVias, F.Cu at (116.5, 115.1)
- added U25: LT3094xDD, Package_DFN_QFN:DFN-12-1EP_3x3mm_P0.45mm_EP1.65x2.38mm_ThermalVias, F.Cu at (116.0, 120.5)
- added U26: TS5A3159DBVR, custom:SOT95P280X145-6N, F.Cu at (165.2, 69.5)
- added U3: TUSB546A-DCIRNQR, custom:RNQ0040A, F.Cu at (107.2, 117.3)
- added U4: BQ25895RTWR, custom:QFN50P400X400X80-25N, F.Cu at (116.7, 108.8)
- added U5: MAX17055ETB_T, custom:SON40P200X250X80-11N, F.Cu at (122.6, 113.7)
- added U6: U_DAC_L, custom:QFN_CS43198_CIR, F.Cu at (165.9, 53.8)
- added U7: U_DAC_R, custom:QFN_CS43198_CIR, F.Cu at (165.9, 61.4)
- added U8: TPS7A2018PDBVR, custom:SOT95P280X145-5N, F.Cu at (172.9, 52.2)
- added U9: TPS7A2033PDBVR, custom:SOT95P280X145-5N, F.Cu at (172.9, 56.7)
