File: a2audio/A2_Audio_Rev1/A2_Audio_Rev1.kicad_sch (KiCad schematic)
At the start: 33 parts, among them J2 AudioJack3, J3 BOOT_JUMPER, SW1 SW_Push, SW2 WIFI_SLIDER, SW3 RotaryEncoder_Switch, SW4 BT_SLIDER, SW5 SW_PREV, SW6 SW_NEXT, SW7 SW_PLAY, U15 CM5108000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

Commit message: Added the new kicad footprints for each schematic, that didn't have one previously (most of them).
Parts:
- U15: footprint CM5108000:MODULE_CM5108000 -> custom:MODULE_CM5108000
- U23: footprint LTC2954ITS8-1_TRPBF:TSOT-23_TS8 -> custom:TSOT-23_TS8
Changed lines of the file:
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@@
 			)
 		)
-		(property "Footprint" "CM5108000:MODULE_CM5108000"
+		(property "Footprint" "custom:MODULE_CM5108000"
 			(at 494.03 228.6 0)
 			(hide yes)
@@
 			)
 		)
-		(property "Footprint" "CM5108000:MODULE_CM5108000"
+		(property "Footprint" "custom:MODULE_CM5108000"
 			(at 347.98 224.79 0)
 			(hide yes)
@@
 			)
 		)
-		(property "Footprint" "LTC2954ITS8-1_TRPBF:TSOT-23_TS8"
+		(property "Footprint" "custom:TSOT-23_TS8"
 			(at 247.65 242.57 0)
 			(hide yes)
