File: a2audio/A2_Audio_Rev1/Audio_Engine.kicad_sch (KiCad schematic)
At the start: 22 parts, among them U10 OPA1622IDRCR, U6 U_DAC_L, U7 U_DAC_R, U8 TPS7A2018PDBVR, U9 TPS7A2033PDBVR

Commit message: Added the new kicad footprints for each schematic, that didn't have one previously (most of them).
Parts:
- U10: footprint OPA1622IDRCR:IC_OPA1622IDRCR -> custom:IC_OPA1622IDRCR
- U6, U7: footprint QFN_CS43198_CIR -> custom:QFN_CS43198_CIR
- U8, U9: footprint TPS7A2033PDBVR:SOT95P280X145-5N -> custom:SOT95P280X145-5N
Changed lines of the file:
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@@
 			)
 		)
-		(property "Footprint" "TPS7A2033PDBVR:SOT95P280X145-5N"
+		(property "Footprint" "custom:SOT95P280X145-5N"
 			(at 185.42 152.4 0)
 			(hide yes)
@@
 			)
 		)
-		(property "Footprint" "QFN_CS43198_CIR"
+		(property "Footprint" "custom:QFN_CS43198_CIR"
 			(at 185.42 44.45 0)
 			(hide yes)
@@
 			)
 		)
-		(property "Footprint" "OPA1622IDRCR:IC_OPA1622IDRCR"
+		(property "Footprint" "custom:IC_OPA1622IDRCR"
 			(at 392.43 133.35 0)
 			(hide yes)
@@
 			)
 		)
-		(property "Footprint" "TPS7A2033PDBVR:SOT95P280X145-5N"
+		(property "Footprint" "custom:SOT95P280X145-5N"
 			(at 246.38 149.86 0)
 			(hide yes)
@@
 			)
 		)
-		(property "Footprint" "QFN_CS43198_CIR"
+		(property "Footprint" "custom:QFN_CS43198_CIR"
 			(at 41.91 44.45 0)
 			(hide yes)
