File: a2audio/A2_Audio_Rev1/Power_Delivery.kicad_sch (KiCad schematic)
At the start: 93 parts, among them J1 USB_C_Receptacle, U1 USBLC6-2SC6, U13 LT3042xMSE, U14 W25Q16JVSS, U19 TPS62130, U2 TPS65987DDHRSHR, U21 TPS61230DRC, U24 TPS65131RGE, U25 LT3094xDD, U3 TUSB546A-DCIRNQR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

Commit message: Added the new kicad footprints for each schematic, that didn't have one previously (most of them).
Parts:
- U2: footprint TPS65987DDHRSHR:IC_TPS65987DDHRSHR -> custom:IC_TPS65987DDHRSHR
- U3: footprint RNQ0040A -> custom:RNQ0040A
- U4: footprint BQ25895RTWR:QFN50P400X400X80-25N -> custom:QFN50P400X400X80-25N
- U5: footprint MAX17055ETB_T:SON40P200X250X80-11N -> custom:SON40P200X250X80-11N
Changed lines of the file:
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@@
 			)
 		)
-		(property "Footprint" "TPS65987DDHRSHR:IC_TPS65987DDHRSHR"
+		(property "Footprint" "custom:IC_TPS65987DDHRSHR"
 			(at 55.88 72.39 0)
 			(hide yes)
@@
 			)
 		)
-		(property "Footprint" "MAX17055ETB_T:SON40P200X250X80-11N"
+		(property "Footprint" "custom:SON40P200X250X80-11N"
 			(at 297.18 201.93 0)
 			(hide yes)
@@
 			)
 		)
-		(property "Footprint" "BQ25895RTWR:QFN50P400X400X80-25N"
+		(property "Footprint" "custom:QFN50P400X400X80-25N"
 			(at 91.44 294.64 0)
 			(hide yes)
@@
 			)
 		)
-		(property "Footprint" "RNQ0040A"
+		(property "Footprint" "custom:RNQ0040A"
 			(at 186.69 111.76 0)
 			(hide yes)
