File: a2audio/A2_Audio_Rev1/Recording&Radio_Engine.kicad_sch (KiCad schematic)
At the start: 28 parts, among them IC1 ES9822QPRO, U11 SI4732-A10-GS, U12 OPA1612AIDR, U16 AP2112K-3.3, U17 AP2112K-1.8, Y1 Crystal

Commit message: Added the new kicad footprints for each schematic, that didn't have one previously (most of them).
Parts:
- IC1: footprint QFN40P500X500X80-41N-D -> custom:QFN40P500X500X80-41N-D
- U11: footprint SOIC_A10-GS_SIL -> custom:SOIC_A10-GS_SIL
- U12: footprint OPA1612AIDR:SOIC127P599X175-8N -> custom:SOIC127P599X175-8N
Changed lines of the file:
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@@
 			)
 		)
-		(property "Footprint" "QFN40P500X500X80-41N-D"
+		(property "Footprint" "custom:QFN40P500X500X80-41N-D"
 			(at 342.9 131.75 0)
 			(hide yes)
@@
 			)
 		)
-		(property "Footprint" "OPA1612AIDR:SOIC127P599X175-8N"
+		(property "Footprint" "custom:SOIC127P599X175-8N"
 			(at 231.14 58.42 0)
 			(hide yes)
@@
 			)
 		)
-		(property "Footprint" "SOIC_A10-GS_SIL"
+		(property "Footprint" "custom:SOIC_A10-GS_SIL"
 			(at 104.14 46.99 0)
 			(hide yes)
