File: a2audio/A2_Audio_Rev1/Video_Engine.kicad_sch (KiCad schematic)
At the start: 21 parts, among them U18 LT6711A, U20 AP2112K-1.8, U22 AP2112K-1.2, Y2 27MHz

Commit message: Added the new kicad footprints for each schematic, that didn't have one previously (most of them).
Parts:
- U18: footprint (none) -> custom:QFN40P750X750X80-65N-D
Changed lines of the file:
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@@
 			)
 		)
-		(property "Footprint" ""
+		(property "Footprint" "custom:QFN40P750X750X80-65N-D"
 			(at 124.46 74.93 0)
 			(hide yes)
