File: a2audio/A2_Audio_Rev1/Vital_Engine.kicad_sch (KiCad schematic)
At the start: 13 parts, among them J4 Micro_SD_Card, J5 Conn_01x15, U26 TS5A3159DBVR

Commit message: Added the new kicad footprints for each schematic, that didn't have one previously (most of them).
Parts:
- U26: footprint TS5A3159DBVR:SOT95P280X145-6N -> custom:SOT95P280X145-6N
Changed lines of the file:
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@@
 			)
 		)
-		(property "Footprint" "TS5A3159DBVR:SOT95P280X145-6N"
+		(property "Footprint" "custom:SOT95P280X145-6N"
 			(at 382.27 87.63 0)
 			(hide yes)
