File: A2Audio_Mainboard/A2_Audio_Rev1/A2_Audio_Rev1.kicad_sch (KiCad schematic)
At the start: 37 parts, among them J3 BOOT_JUMPER, J7 SJ2-35954B-SMT-TR, SW1 SW_Wuerth_450301014042, SW10 EVQ-PUJ02K, SW11 EVQ-PUJ02K, SW3 RotaryEncoder_Switch, SW4 SW_Wuerth_450301014042, SW8 EVQ-PUJ02K, SW9 EVQ-PUJ02K, U15 CM5108000, U23 LTC2954ITS8-1_TRPBF

Commit message: Fixed even more schematic errors
Connections:
- net CARD_DETECT: now also U15.37 (GPIO7); no longer U15.31 (GPIO12)
- net I2C_SCL_AUDIO: now reaches U15.28 (GPIO13)
- new net I2C_SDA_AUDIO: U15.31 (GPIO12)
Other:
- sheet Recording&Radio_Engine ports: added I2C_SCL_AUDIO, I2C_SDA_AUDIO; removed none
Changed lines of the file:
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@@
 	(wire
 		(pts
+			(xy 43.18 218.44) (xy 64.77 218.44)
+		)
+		(stroke
+			(width 0)
+			(type default)
+		)
+	)
+	(wire
+		(pts
 			(xy 434.34 326.39) (xy 434.34 297.18)
 		)
@@
 	(wire
 		(pts
+			(xy 378.46 224.79) (xy 396.24 224.79)
+		)
+		(stroke
+			(width 0)
+			(type default)
+		)
+	)
+	(wire
+		(pts
 			(xy 162.56 265.43) (xy 162.56 382.27)
 		)
@@
 	(wire
 		(pts
+			(xy 43.18 220.98) (xy 64.77 220.98)
+		)
+		(stroke
+			(width 0)
+			(type default)
+		)
+	)
+	(wire
+		(pts
 			(xy 172.72 80.01) (xy 172.72 78.74)
 		)
@@
 	(wire
 		(pts
+			(xy 378.46 227.33) (xy 396.24 227.33)
+		)
+		(stroke
+			(width 0)
+			(type default)
+		)
+	)
+	(wire
+		(pts
 			(xy 509.27 82.55) (xy 513.08 82.55)
 		)
@@
 	)
 	(label "CARD_DETECT"
-		(at 378.46 224.79 0)
+		(at 378.46 212.09 0)
 		(effects
 			(font
@@
 		)
 	)
-	(label "I2C_SDA"
+	(label "I2C_SDA_AUDIO"
 		(at 49.53 80.01 0)
 		(effects
@@
 		)
 	)
+	(label "I2C_SCL_AUDIO"
+		(at 43.18 218.44 0)
+		(effects
+			(font
+				(size 1.27 1.27)
+			)
+			(justify left bottom)
+		)
+	)
 	(label "+5V"
 		(at 232.41 227.33 0)
@@
 		)
 	)
+	(label "I2C_SDA_AUDIO"
+		(at 396.24 224.79 0)
+		(effects
+			(font
+				(size 1.27 1.27)
+			)
+			(justify left bottom)
+		)
+	)
 	(label "SCL"
 		(at 307.34 102.87 0)
@@
 		)
 	)
+	(label "I2C_SCL_AUDIO"
+		(at 396.24 227.33 0)
+		(effects
+			(font
+				(size 1.27 1.27)
+			)
+			(justify left bottom)
+		)
+	)
 	(label "HP_DETECT"
 		(at 378.46 229.87 0)
@@
 		)
 	)
-	(label "I2C_SCL"
+	(label "I2C_SCL_AUDIO"
 		(at 49.53 83.82 0)
 		(effects
@@
 		)
 	)
+	(label "I2C_SDA_AUDIO"
+		(at 43.18 220.98 0)
+		(effects
+			(font
+				(size 1.27 1.27)
+			)
+			(justify left bottom)
+		)
+	)
 	(label "SD_DAT2"
 		(at 275.59 88.9 180)
@@
 			(effects
 				(font
+					(size 1.27 1.27)
+				)
+				(justify left)
+			)
+		)
+		(pin "I2C_SCL_AUDIO" bidirectional
+			(at 64.77 218.44 180)
+			(effects
+				(font
+					(size 1.27 1.27)
+				)
+				(justify left)
+			)
+		)
+		(pin "I2C_SDA_AUDIO" bidirectional
+			(at 64.77 220.98 180)
+			(effects
+				(font

Commit message: Final touches in schematic
Other:
- sheet Vital_Engine ports: added none; removed +5V_DSI
Changed lines of the file:
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@@
 		)
 	)
-	(label "+5V"
-		(at 307.34 106.68 0)
-		(effects
-			(font
-				(size 1.27 1.27)
-			)
-			(justify left bottom)
-		)
-	)
 	(label "ENC_1"
 		(at 505.46 66.04 180)
@@
 			(effects
 				(font
-					(size 1.27 1.27)
-				)
-				(justify right)
-			)
-		)
-		(pin "+5V_DSI" input
-			(at 307.34 106.68 0)
-			(effects
-				(font

Commit message: Fixed SD Card logic and power error
Parts:
- SW3: footprint (none) -> custom:XDCR_RING35-203010-TH
Connections:
- net +3V3_SYS: no longer R29.1, R30.1, R41.2, R42.1, R43.2, R44.1, R45.1, R46.1, R47.1, R48.1, R49.1, R54.2
- net CM5_3.3V(OUTPUT): now also R29.1, R30.1, R41.2, R42.1, R43.2, R44.1, R45.1, R46.1, R47.1, R48.1, R49.1, R54.2, U15.78 (GPIO_VREF)
- net SD_PWRON: now reaches U15.75 (SD_PWR_ON)
- net VDD_OVERRIDE: no longer names the net of U15.73 (SD_VDD_OVERRIDE)
Other:
- sheet Power&Battery ports: added +3V3_SYSPI; removed none
- sheet Vital_Engine ports: added 3V3_PI, CM5_CD, SD_PWR_ONCM5; removed +1V8_SD, CARD_DETECT, SD_VDD_OVERRIDE
